Commit message: feat: describe the wheel shafts and ultrasonic rangers in the URDF
Four shafts and four rangers existed only as meshes the visualiser drew onto
the scene topic, so this description covered five of the vehicle's thirteen
visible parts. Their transforms were already published; only the links were
missing, which is why the gap was invisible until something tried to render the
robot from its description alone.

Poses are the visualiser's own constants, transcribed unchanged.

Co-Authored-By: Claude Opus 5 (1M context) <noreply@anthropic.com>
Claude-Session: https://claude.ai/code/session_01PTgpaexUo6cTtJmKkbi552

File: urdf/mecanum_visual.urdf (robot description, URDF)
Before this commit: robot xgc2_mecanum_ugv, 6 links, 5 joints
Links:
- added link front_sensor; visual mesh filename=package://mecanum_description/meshes/urm04.STL
- added link left_sensor; visual mesh filename=package://mecanum_description/meshes/urm04.STL
- added link lower_left_wheel_shaft; visual mesh filename=package://mecanum_description/meshes/wheel_shaft.STL
- added link lower_right_wheel_shaft; visual mesh filename=package://mecanum_description/meshes/wheel_shaft.STL
- added link rear_sensor; visual mesh filename=package://mecanum_description/meshes/urm04.STL
- added link right_sensor; visual mesh filename=package://mecanum_description/meshes/urm04.STL
- added link upper_left_wheel_shaft; visual mesh filename=package://mecanum_description/meshes/wheel_shaft.STL
- added link upper_right_wheel_shaft; visual mesh filename=package://mecanum_description/meshes/wheel_shaft.STL
Joints:
- added joint front_sensor_joint: type fixed, parent base_link, child front_sensor, origin xyz=0.205 0 0.06 rpy=1.5707963267948966 0 0
- added joint left_sensor_joint: type fixed, parent base_link, child left_sensor, origin xyz=0 0.108 0.06 rpy=1.5707963267948966 0 1.5707963267948966
- added joint lower_left_wheel_shaft_joint: type fixed, parent base_link, child lower_left_wheel_shaft, origin xyz=-0.150 0.108 0.05 rpy=0 0 0
- added joint lower_right_wheel_shaft_joint: type fixed, parent base_link, child lower_right_wheel_shaft, origin xyz=-0.150 -0.108 0.05 rpy=3.141592653589793 0 0
- added joint rear_sensor_joint: type fixed, parent base_link, child rear_sensor, origin xyz=-0.201 0 0.06 rpy=1.5707963267948966 0 3.141592653589793
- added joint right_sensor_joint: type fixed, parent base_link, child right_sensor, origin xyz=0 -0.108 0.06 rpy=1.5707963267948966 0 -1.5707963267948966
- added joint upper_left_wheel_shaft_joint: type fixed, parent base_link, child upper_left_wheel_shaft, origin xyz=0.150 0.108 0.05 rpy=0 0 0
- added joint upper_right_wheel_shaft_joint: type fixed, parent base_link, child upper_right_wheel_shaft, origin xyz=0.150 -0.108 0.05 rpy=3.141592653589793 0 0
