Commit message: fix: align Mecanum viewer URDF with Gazebo

File: urdf/mecanum_visual.urdf (robot description, URDF)
Before this commit: robot xgc2_mecanum_ugv, 14 links, 13 joints
Links:
- removed link base_footprint
- link base_link: geometry visual box size=0.02 0.08 0.01; visual mesh filename=package://mecanum_description/meshes/nexus_base_link.STL scale=0.001 0.001 0.001
- link front_sensor: geometry visual mesh filename=package://mecanum_description/meshes/urm04.STL scale=0.001 0.001 0.001
- link left_sensor: geometry visual mesh filename=package://mecanum_description/meshes/urm04.STL scale=0.001 0.001 0.001
- link lower_left_wheel_shaft: geometry visual mesh filename=package://mecanum_description/meshes/wheel_shaft.STL scale=0.001 0.001 0.001
- link lower_right_wheel_shaft: geometry visual mesh filename=package://mecanum_description/meshes/wheel_shaft.STL scale=0.001 0.001 0.001
- link rear_sensor: geometry visual mesh filename=package://mecanum_description/meshes/urm04.STL scale=0.001 0.001 0.001
- link right_sensor: geometry visual mesh filename=package://mecanum_description/meshes/urm04.STL scale=0.001 0.001 0.001
- link upper_left_wheel_shaft: geometry visual mesh filename=package://mecanum_description/meshes/wheel_shaft.STL scale=0.001 0.001 0.001
- link upper_right_wheel_shaft: geometry visual mesh filename=package://mecanum_description/meshes/wheel_shaft.STL scale=0.001 0.001 0.001
Joints:
- removed joint base_joint
- joint lower_left_wheel_joint: axis 0 1 0 -> (none); parent base_footprint -> base_link; type continuous -> fixed
- joint lower_right_wheel_joint: axis 0 1 0 -> (none); parent base_footprint -> base_link; type continuous -> fixed
- joint upper_left_wheel_joint: axis 0 1 0 -> (none); parent base_footprint -> base_link; type continuous -> fixed
- joint upper_right_wheel_joint: axis 0 1 0 -> (none); parent base_footprint -> base_link; type continuous -> fixed
